File: HW-nums/nums.sch (KiCad schematic (older format))
At the start: 64 parts, among them CON101 AVR-ISP-6, IC101 ATMEGA88A-A, P101 CONN_2, Q101 MOSFET_N, Q102 MOSFET_N, Q103 MOSFET_N, U101 MC34063, U102 AD5700, U103 OPA690, X101 QUARTZCMS4

Commit message: update
Connections:
- net PWR2: now reaches C101.1, FB101.2, R101.1, R102.1, R104.1, U101.6 (VCC)
- net PWR3: now reaches R101.2, R102.2, R104.2, U101.1 (Sw_Coll), U101.7 (I_Sense), U101.8 (Drv_Coll)
- net PWR4: now reaches D102.2 (K), L101.1, U101.2 (Sw_Emit)
- net PWR1: now reaches FB101.1, R103.2
- net RE: now reaches R111.2, S101.1 (Segm_E), S102.1 (Segm_E), S103.1 (Segm_E)
- net RG: now reaches R113.2, S101.10 (Segm_G), S102.10 (Segm_G), S103.10 (Segm_G)
- net RD: now reaches R110.2, S101.2 (Segm_D), S102.2 (Segm_D), S103.2 (Segm_D)
- net K0: now reaches Q101.D, S101.3 (K), S101.8 (K)
- net RC: now reaches R109.2, S101.4 (Segm_C), S102.4 (Segm_C), S103.4 (Segm_C)
- net RDP: now reaches R114.2, S101.5 (SegmDP), S102.5 (SegmDP), S103.5 (SegmDP)
- net RB: now reaches R108.2, S101.6 (Segm_B), S102.6 (Segm_B), S103.6 (Segm_B)
- net RA: now reaches R107.2, S101.7 (Segm_A), S102.7 (Segm_A), S103.7 (Segm_A)
- net RF: now reaches R112.2, S101.9 (Segm_F), S102.9 (Segm_F), S103.9 (Segm_F)
- net K1: now reaches Q102.D, S102.3 (K), S102.8 (K)
- net K2: now reaches Q103.D, S103.3 (K), S103.8 (K)

Commit message: update
Connections:
- net A: now also IC101.11 ((PCINT23/AIN1)PD7); no longer IC101.12 ((PCINT0/CLKO/ICP1)PB0)
- net B: now also IC101.12 ((PCINT0/CLKO/ICP1)PB0); no longer IC101.13 ((PCINT1/OC1A)PB1)
- net C: now also IC101.15 ((PCINT3/OC2A/MOSI)PB3); no longer IC101.23 ((PCINT8/ADC0)PC0)
- net D: now also IC101.16 ((PCINT4/MISO)PB4); no longer CON101.3, IC101.17 ((PCINT5/SCK)PB5)
- net DP: now also IC101.23 ((PCINT8/ADC0)PC0); no longer IC101.24 ((PCINT9/ADC1)PC1)
- net E: now also IC101.17 ((PCINT5/SCK)PB5); no longer CON101.1, IC101.16 ((PCINT4/MISO)PB4)
- net F: now also IC101.13 ((PCINT1/OC1A)PB1); no longer IC101.14 ((PCINT2/OC1B/SS)PB2)
- net G: now also IC101.14 ((PCINT2/OC1B/SS)PB2); no longer CON101.4, IC101.15 ((PCINT3/OC2A/MOSI)PB3)
- net RC: now also CON101.4
- net RD: now also CON101.1
- net RE: now also CON101.3
- net seg0: now also R115.2
- net seg1: now also R116.2
- net seg2: now also R117.2
- no-connect marks 3 -> 4
